File: HW/SBC_multisheet/acia_max232.sch (KiCad schematic (older format))
At the start: 0 parts

Commit message: PLUTO SBC with RTC schematics done.
Parts:
- added C1, C2, C4: 10uF, symbol CP1_Small
- added C3, C5: 4.7uF, symbol CP1_Small
- added C6: 22pF, symbol C_Small
- added J1: Serial Port, symbol CONN_02X05
- added Pad1: RI, symbol Mounting_Hole_PAD
- added U4: MAX232, symbol MAX232
- added U5: 6551, symbol 6551
- added XTAL1: 1.8432 MHz, symbol CRYSTAL
Connections:
- new net: U4.10 (T2IN), U5.10 (TxD)
- new net: U4.9 (R2OUT), U5.12 (RxD)
- new net: C6.1, U5.6 (XTLI), XTAL1.1
- new net: U5.7 (XTLO), XTAL1.2
- new net: U4.11 (T1IN), U5.8 (~RTS)
- new net: U4.12 (R1OUT), U5.9 (~CTS)
- new net: C5.1, U4.1 (C1+)
- new net: J1.8 (P8), U4.13 (R1IN)
- new net: J1.7 (P7), U4.14 (T1OUT)
- new net: C2.1, U4.2 (VS+)
- new net: C5.2, U4.3 (C1-)
- new net: C3.1, U4.4 (C2+)
- new net: C3.2, U4.5 (C2-)
- new net: C1.2, U4.6 (VS-)
- new net: J1.3 (P3), U4.7 (T2OUT)
- new net: J1.2 (P2), U4.8 (R2IN)
- new net: J1.9 (P9), Pad1.1
- new net A0: U5.13 (RS0)
- new net A1: U5.14 (RS1)
- new net CLK: U5.27 (PHI2-IN)
- new net D0: U5.18 (D0)
- new net D1: U5.19 (D1)
- new net D2: U5.20 (D2)
- new net D3: U5.21 (D3)
- new net D4: U5.22 (D4)
- new net D5: U5.23 (D5)
- new net D6: U5.24 (D6)
- new net D7: U5.25 (D7)
- new net GND: C1.1, C4.2, C6.2, J1.5 (P5), U4.15 (GND), U5.16 (~DCD), U5.17 (~DSR)
- new net R/~W: U5.28 (R/~W)
- new net VCC: C2.2, C4.1, U4.16 (VCC), U5.2 (CS1)
- new net ~7FEX: U5.3 (~CS2)
- new net ~IRQ: U5.26 (~IRQ)
- new net ~RES: U5.4 (~RES)
- no-connect marks 0 -> 6

Commit message: The PCB layout editor doesn't like 7805's footprint.
Parts:
- C1, C2, C3, C4, C5: footprint (none) -> Capacitors_ThroughHole:CP_Radial_D5.0mm_P2.50mm
- C6: footprint (none) -> Capacitors_ThroughHole:C_Disc_D3.8mm_W2.6mm_P2.50mm
- J1: footprint (none) -> Pin_Headers:Pin_Header_Straight_2x05_Pitch2.54mm
- Pad1: footprint (none) -> Wire_Pads:SolderWirePad_single_0-8mmDrill
- U4: footprint (none) -> Housings_DIP:DIP-16_W7.62mm
- U5: footprint (none) -> Housings_DIP:DIP-28_W15.24mm
- XTAL1: footprint (none) -> Crystals:Resonator-2pin_w10.0mm_h5.0mm
Connections:
- net GND: now also U5.1 (GND)
- net VCC: now also U5.15 (VCC)
Changed lines of the file:
@@
 F 0 "U5" H 7750 4475 60  0000 C CNN
 F 1 "6551" V 7975 3150 60  0000 C CNN
-F 2 "" H 8025 2475 60  0001 C CNN
+F 2 "Housings_DIP:DIP-28_W15.24mm" H 8025 2475 60  0001 C CNN
 F 3 "" H 8025 2475 60  0001 C CNN
 	1    7975 3150
@@
 F 0 "U4" H 4950 2075 50  0000 R CNN
 F 1 "MAX232" H 4400 4200 50  0000 R CNN
-F 2 "" H 4550 2100 50  0001 L CNN
+F 2 "Housings_DIP:DIP-16_W7.62mm" H 4550 2100 50  0001 L CNN
 F 3 "" H 4500 3250 50  0001 C CNN
 	1    4500 3150
@@
 A1
 $Comp
-L VCC #PWR9
+L VCC #PWR01
 U 1 1 58D6F59A
 P 9500 3475
-F 0 "#PWR9" H 9500 3325 50  0001 C CNN
+F 0 "#PWR01" H 9500 3325 50  0001 C CNN
 F 1 "VCC" H 9500 3625 50  0000 C CNN
 F 2 "" H 9500 3475 50  0001 C CNN
@@
 F 0 "XTAL1" V 6900 2250 60  0000 C CNN
 F 1 "1.8432 MHz" V 6750 2050 60  0000 C CNN
-F 2 "" H 6825 2050 60  0001 C CNN
+F 2 "Crystals:Resonator-2pin_w10.0mm_h5.0mm" H 6825 2050 60  0001 C CNN
 F 3 "" H 6925 2150 60  0001 C CNN
 	1    6925 2050
@@
 F 0 "C6" H 6550 2100 50  0000 L CNN
 F 1 "22pF" H 6200 2125 50  0000 L CNN
-F 2 "" H 6450 2050 50  0001 C CNN
+F 2 "Capacitors_ThroughHole:C_Disc_D3.8mm_W2.6mm_P2.50mm" H 6450 2050 50  0001 C CNN
 F 3 "" H 6450 2050 50  0001 C CNN
 	1    6450 2050
@@
 $EndComp
 $Comp
-L GND #PWR6
+L GND #PWR02
 U 1 1 58D7044A
 P 6450 2150
-F 0 "#PWR6" H 6450 1900 50  0001 C CNN
+F 0 "#PWR02" H 6450 1900 50  0001 C CNN
 F 1 "GND" H 6450 2000 50  0000 C CNN
 F 2 "" H 6450 2150 50  0001 C CNN
@@
 F 0 "C3" H 3650 3900 50  0000 L CNN
 F 1 "4.7uF" H 3650 4050 50  0000 L CNN
-F 2 "" H 3575 3950 50  0001 C CNN
+F 2 "Capacitors_ThroughHole:CP_Radial_D5.0mm_P2.50mm" H 3575 3950 50  0001 C CNN
 F 3 "" H 3575 3950 50  0001 C CNN
 	1    3575 3950
@@
 F 0 "C2" V 3425 3375 50  0000 L CNN
 F 1 "10uF" V 3600 3325 50  0000 L CNN
-F 2 "" H 3475 3550 50  0001 C CNN
+F 2 "Capacitors_ThroughHole:CP_Radial_D5.0mm_P2.50mm" H 3475 3550 50  0001 C CNN
 F 3 "" H 3475 3550 50  0001 C CNN
 	1    3475 3550
@@
 F 0 "C1" V 3550 3325 50  0000 L CNN
 F 1 "10uF" V 3350 3275 50  0000 L CNN
-F 2 "" H 3475 3250 50  0001 C CNN
+F 2 "Capacitors_ThroughHole:CP_Radial_D5.0mm_P2.50mm" H 3475 3250 50  0001 C CNN
 F 3 "" H 3475 3250 50  0001 C CNN
 	1    3475 3250
@@
 F 0 "C4" H 4935 4670 50  0000 L CNN
 F 1 "10uF" H 4935 4520 50  0000 L CNN
-F 2 "" H 4925 4600 50  0001 C CNN
+F 2 "Capacitors_ThroughHole:CP_Radial_D5.0mm_P2.50mm" H 4925 4600 50  0001 C CNN
 F 3 "" H 4925 4600 50  0001 C CNN
 	1    4925 4600
@@
 F 0 "C5" H 5275 3875 50  0000 L CNN
 F 1 "4.7uF" H 5150 4025 50  0000 L CNN
-F 2 "" H 5425 3950 50  0001 C CNN
+F 2 "Capacitors_ThroughHole:CP_Radial_D5.0mm_P2.50mm" H 5425 3950 50  0001 C CNN
 F 3 "" H 5425 3950 50  0001 C CNN
 	1    5425 3950
@@
 $EndComp
 $Comp
-L GND #PWR2
+L GND #PWR03
 U 1 1 58D716F3
 P 3050 3250
-F 0 "#PWR2" H 3050 3000 50  0001 C CNN
+F 0 "#PWR03" H 3050 3000 50  0001 C CNN
 F 1 "GND" H 3050 3100 50  0000 C CNN
 F 2 "" H 3050 3250 50  0001 C CNN
@@
 $EndComp
 $Comp
-L VCC #PWR4
+L VCC #PWR04
 U 1 1 58D7177E
 P 4500 4625
-F 0 "#PWR4" H 4500 4475 50  0001 C CNN
+F 0 "#PWR04" H 4500 4475 50  0001 C CNN
 F 1 "VCC" H 4500 4775 50  0000 C CNN
 F 2 "" H 4500 4625 50  0001 C CNN
@@
 F 0 "J1" H 2075 2950 50  0000 C CNN
 F 1 "Serial Port" H 2075 2350 50  0000 C CNN
-F 2 "" H 2075 1450 50  0001 C CNN
+F 2 "Pin_Headers:Pin_Header_Straight_2x05_Pitch2.54mm" H 2075 1450 50  0001 C CNN
 F 3 "" H 2075 1450 50  0001 C CNN
 	1    2075 2650
@@
 $EndComp
 $Comp
-L GND #PWR1
+L GND #PWR05
 U 1 1 58D71F12
 P 1650 3150
-F 0 "#PWR1" H 1650 2900 50  0001 C CNN
+F 0 "#PWR05" H 1650 2900 50  0001 C CNN
 F 1 "GND" H 1650 3000 50  0000 C CNN
 F 2 "" H 1650 3150 50  0001 C CNN
@@
 F 0 "Pad1" H 1475 3450 50  0000 C CNN
 F 1 "RI" H 1475 3375 50  0000 C CNN
-F 2 "" H 1475 3200 50  0001 C CNN
+F 2 "Wire_Pads:SolderWirePad_single_0-8mmDrill" H 1475 3200 50  0001 C CNN
 F 3 "" H 1475 3200 50  0001 C CNN
 	1    1475 3200
@@
 $EndComp
 $Comp
-L GND #PWR5
+L GND #PWR06
 U 1 1 58D72DB3
 P 4925 4700
-F 0 "#PWR5" H 4925 4450 50  0001 C CNN
+F 0 "#PWR06" H 4925 4450 50  0001 C CNN
 F 1 "GND" H 4925 4550 50  0000 C CNN
 F 2 "" H 4925 4700 50  0001 C CNN
@@
 $EndComp
 $Comp
-L GND #PWR3
+L GND #PWR07
 U 1 1 58D73252
 P 4500 1950
-F 0 "#PWR3" H 4500 1700 50  0001 C CNN
+F 0 "#PWR07" H 4500 1700 50  0001 C CNN
 F 1 "GND" H 4500 1800 50  0000 C CNN
 F 2 "" H 4500 1950 50  0001 C CNN
@@
 	6650 2550 6650 2300
 $Comp
-L GND #PWR8
+L GND #PWR08
 U 1 1 58D744C7
 P 7275 3925
-F 0 "#PWR8" H 7275 3675 50  0001 C CNN
+F 0 "#PWR08" H 7275 3675 50  0001 C CNN
 F 1 "GND" H 7275 3775 50  0000 C CNN
 F 2 "" H 7275 3925 50  0001 C CNN
@@
 $EndComp
 $Comp
-L GND #PWR7
+L GND #PWR09
 U 1 1 58D74507
 P 7275 3500
-F 0 "#PWR7" H 7275 3250 50  0001 C CNN
+F 0 "#PWR09" H 7275 3250 50  0001 C CNN
 F 1 "GND" H 7275 3350 50  0000 C CNN
 F 2 "" H 7275 3500 50  0001 C CNN
@@
 NoConn ~ 7275 3275
 NoConn ~ 7275 4175
+$Comp
+L GND #PWR010
+U 1 1 58D84381
+P 7975 4800
+F 0 "#PWR010" H 7975 4550 50  0001 C CNN
+F 1 "GND" H 7975 4650 50  0000 C CNN
+F 2 "" H 7975 4800 50  0001 C CNN
+F 3 "" H 7975 4800 50  0001 C CNN
+	1    7975 4800
+	1    0    0    -1
+$EndComp
+$Comp
+L VCC #PWR011
+U 1 1 58D845E7
+P 7975 1600
+F 0 "#PWR011" H 7975 1450 50  0001 C CNN
+F 1 "VCC" H 7975 1750 50  0000 C CNN
+F 2 "" H 7975 1600 50  0001 C CNN
+F 3 "" H 7975 1600 50  0001 C CNN
+	1    7975 1600
+	1    0    0    -1
+$EndComp
+Wire Wire Line
+	7975 4675 7975 4800
 $EndSCHEMATC
