File: HW/SBC_multisheet/address_decoding_and_support.sch (KiCad schematic (older format))
At the start: 7 parts

Commit message: PLUTO SBC with RTC schematics done.
Parts:
- removed RN?: 3.3kOhm, Resistors_THT:R_Array_SIP6, symbol R_Network05
- added Q1: DS1813, symbol Q_NPN_EBC
- added RN1: 3.3 kOhm, Resistors_THT:R_Array_SIP8, symbol R_Network07
- added SW1: RESET, symbol SW_Push
- added X1: 4 MHz, Oscillators:Oscillator_DIP-8, symbol CXO_DIP8
- gave numbers to parts that had none: 3
Connections:
- net BE: now also RN1.6 (R5)
- net CLK: now also U8.10; no longer U8.13
- net GND: now also Q1.3 (C), SW1.1, X1.4 (GND)
- net R/~W: now also U8.4, U8.5; no longer U8.10, U8.9
- net RDY: now also RN1.4 (R3)
- net VCC: now also Q1.2 (B), RN1.1 (common), X1.8 (Vcc)
- net ~IOSEL: now also U8.13; no longer U8.5
- net ~IRQ: now also RN1.8 (R7)
- net ~MRD: now also U8.6, U8.9; no longer U8.12, U8.8
- net ~MWR: now also U8.8; no longer U8.11
- net ~NMI: now also RN1.7 (R6)
- net ~RAMSEL: now also U8.11; no longer U8.6
- net ~RES: now also Q1.1 (E), RN1.3 (R2), SW1.2
- net ~ROMSEL: now also U8.12; no longer U8.4
- new net PHI2: X1.5 (OUT)
- new net ~PWR: RN1.5 (R4)
- no-connect marks 0 -> 1

Commit message: The PCB layout editor doesn't like 7805's footprint.
Parts:
- Q1: footprint (none) -> TO_SOT_Packages_THT:TO-92_Inline_Narrow_Oval
- RN1: footprint Resistors_THT:R_Array_SIP8 -> Pin_Headers:Pin_Header_Straight_1x08_Pitch2.54mm
- SW1: footprint (none) -> Buttons_Switches_ThroughHole:SW_PUSH_6mm_h4.3mm
- U10: footprint (none) -> Housings_DIP:DIP-16_W7.62mm
- U8, U9: footprint (none) -> Housings_DIP:DIP-14_W7.62mm
Connections:
- no-connect marks 1 -> 2
Changed lines of the file:
@@
 F 0 "U8" H 5450 2200 50  0000 C CNN
 F 1 "74HCT00" H 5450 2050 50  0000 C CNN
-F 2 "" H 5450 2150 50  0001 C CNN
+F 2 "Housings_DIP:DIP-14_W7.62mm" H 5450 2150 50  0001 C CNN
 F 3 "" H 5450 2150 50  0001 C CNN
 	1    5450 2150
@@
 F 0 "U8" H 8150 2650 50  0000 C CNN
 F 1 "74HCT00" H 8150 2500 50  0000 C CNN
-F 2 "" H 8150 2600 50  0001 C CNN
+F 2 "Housings_DIP:DIP-14_W7.62mm" H 8150 2600 50  0001 C CNN
 F 3 "" H 8150 2600 50  0001 C CNN
 	4    8150 2600
@@
 F 0 "U8" H 6250 1250 50  0000 C CNN
 F 1 "74HCT00" H 6250 1100 50  0000 C CNN
-F 2 "" H 6250 1200 50  0001 C CNN
+F 2 "Housings_DIP:DIP-14_W7.62mm" H 6250 1200 50  0001 C CNN
 F 3 "" H 6250 1200 50  0001 C CNN
 	2    6250 1200
@@
 F 0 "U8" H 7800 1725 50  0000 C CNN
 F 1 "74HCT00" H 7800 1575 50  0000 C CNN
-F 2 "" H 7800 1675 50  0001 C CNN
+F 2 "Housings_DIP:DIP-14_W7.62mm" H 7800 1675 50  0001 C CNN
 F 3 "" H 7800 1675 50  0001 C CNN
 	3    7800 1675
@@
 F 0 "U9" H 6950 3175 50  0000 C CNN
 F 1 "74LS30" H 6950 2975 50  0000 C CNN
-F 2 "" H 6950 3075 50  0001 C CNN
+F 2 "Housings_DIP:DIP-14_W7.62mm" H 6950 3075 50  0001 C CNN
 F 3 "" H 6950 3075 50  0001 C CNN
 	1    6950 3075
@@
 F 0 "U10" H 7725 5075 50  0000 C CNN
 F 1 "74LS138" H 8075 4026 50  0000 C CNN
-F 2 "" H 7925 4575 50  0001 C CNN
+F 2 "Housings_DIP:DIP-16_W7.62mm" H 7925 4575 50  0001 C CNN
 F 3 "" H 7925 4575 50  0001 C CNN
 	1    7925 4575
@@
 Text GLabel 9125 5125 2    60   Input ~ 0
 ~7FEX
-Text GLabel 6700 4900 0    60   Input ~ 0
-GND
-Text GLabel 6700 4725 0    60   Input ~ 0
-VCC
 Wire Wire Line
 	6050 2150 9075 2150
@@
 F 0 "RN1" V 1575 1475 50  0000 C CNN
 F 1 "3.3 kOhm" V 2375 1475 50  0000 C CNN
-F 2 "Resistors_THT:R_Array_SIP8" V 2450 1475 50  0001 C CNN
+F 2 "Pin_Headers:Pin_Header_Straight_1x08_Pitch2.54mm" V 2450 1475 50  0001 C CNN
 F 3 "" H 1975 1475 50  0001 C CNN
 	1    1975 1475
@@
 PHI2
 $Comp
-L VCC #PWR19
+L VCC #PWR021
 U 1 1 58D6CEDE
 P 1875 4350
-F 0 "#PWR19" H 1875 4200 50  0001 C CNN
+F 0 "#PWR021" H 1875 4200 50  0001 C CNN
 F 1 "VCC" H 1875 4500 50  0000 C CNN
 F 2 "" H 1875 4350 50  0001 C CNN
@@
 $EndComp
 $Comp
-L GND #PWR20
+L GND #PWR022
 U 1 1 58D6CF02
 P 1875 4950
-F 0 "#PWR20" H 1875 4700 50  0001 C CNN
+F 0 "#PWR022" H 1875 4700 50  0001 C CNN
 F 1 "GND" H 1875 4800 50  0000 C CNN
 F 2 "" H 1875 4950 50  0001 C CNN
@@
 F 0 "Q1" H 1775 2850 50  0000 L CNN
 F 1 "DS1813" H 1550 3200 50  0000 L CNN
-F 2 "" H 2075 3125 50  0001 C CNN
+F 2 "TO_SOT_Packages_THT:TO-92_Inline_Narrow_Oval" H 2075 3125 50  0001 C CNN
 F 3 "" H 1875 3025 50  0001 C CNN
 	1    1875 3025
@@
 $EndComp
 $Comp
-L VCC #PWR21
+L VCC #PWR023
 U 1 1 58D6D2F3
 P 2075 3025
-F 0 "#PWR21" H 2075 2875 50  0001 C CNN
+F 0 "#PWR023" H 2075 2875 50  0001 C CNN
 F 1 "VCC" H 2075 3175 50  0000 C CNN
 F 2 "" H 2075 3025 50  0001 C CNN
@@
 F 0 "SW1" H 1050 2725 50  0000 L CNN
 F 1 "RESET" H 1125 3000 50  0000 C CNN
-F 2 "" H 1125 3025 50  0001 C CNN
+F 2 "Buttons_Switches_ThroughHole:SW_PUSH_6mm_h4.3mm" H 1125 3025 50  0001 C CNN
 F 3 "" H 1125 3025 50  0001 C CNN
 	1    1125 2825
@@
 	1775 3225 1775 3400
 $Comp
-L GND #PWR18
+L GND #PWR024
 U 1 1 58D6D657
 P 1775 3400
-F 0 "#PWR18" H 1775 3150 50  0001 C CNN
+F 0 "#PWR024" H 1775 3150 50  0001 C CNN
 F 1 "GND" H 1775 3250 50  0000 C CNN
 F 2 "" H 1775 3400 50  0001 C CNN
@@
 Connection ~ 1775 2650
 $Comp
-L VCC #PWR17
+L VCC #PWR025
 U 1 1 58D7E610
 P 1675 1100
-F 0 "#PWR17" H 1675 950 50  0001 C CNN
+F 0 "#PWR025" H 1675 950 50  0001 C CNN
 F 1 "VCC" H 1675 1250 50  0000 C CNN
 F 2 "" H 1675 1100 50  0001 C CNN
@@
 	1    0    0    -1
 $EndComp
+$Comp
+L VCC #PWR026
+U 1 1 58D83088
+P 6700 4725
+F 0 "#PWR026" H 6700 4575 50  0001 C CNN
+F 1 "VCC" H 6700 4875 50  0000 C CNN
+F 2 "" H 6700 4725 50  0001 C CNN
+F 3 "" H 6700 4725 50  0001 C CNN
+	1    6700 4725
+	0    -1   -1   0
+$EndComp
+$Comp
+L GND #PWR027
+U 1 1 58D830F6
+P 6700 4900
+F 0 "#PWR027" H 6700 4650 50  0001 C CNN
+F 1 "GND" H 6700 4750 50  0000 C CNN
+F 2 "" H 6700 4900 50  0001 C CNN
+F 3 "" H 6700 4900 50  0001 C CNN
+	1    6700 4900
+	0    1    1    0
+$EndComp
+NoConn ~ 1675 1675
 $EndSCHEMATC
