File: HW/SBC_multisheet/via_rtc.sch (KiCad schematic (older format))
At the start: 0 parts

Commit message: PLUTO SBC with RTC schematics done.
Parts:
- added D1: D, symbol D_Small
- added J2, J3: CONN_02X07, symbol CONN_02X07
- added U6: WD65C22, symbol WD65C22
- added U7: DS1511Y+, symbol DS1511Y+
Connections:
- new net: J3.3 (P3), U6.10 (PB0)
- new net: J3.4 (P4), U6.11 (PB1)
- new net: J3.5 (P5), U6.12 (PB2)
- new net: J3.6 (P6), U6.13 (PB3)
- new net: J3.7 (P7), U6.14 (PB4)
- new net: J3.8 (P8), U6.15 (PB5)
- new net: J3.9 (P9), U6.16 (PB6)
- new net: J3.10 (P10), U6.17 (PB7)
- new net: J3.11 (P11), U6.18 (CB1)
- new net: J3.12 (P12), U6.19 (CB2)
- new net: J2.3 (P3), U6.2 (PA0)
- new net: D1.1 (K), U6.21 (~IRQ)
- new net: J2.4 (P4), U6.3 (PA1)
- new net: J2.12 (P12), U6.39 (CA2)
- new net: J2.5 (P5), U6.4 (PA2)
- new net: J2.11 (P11), U6.40 (CA1)
- new net: J2.6 (P6), U6.5 (PA3)
- new net: J2.7 (P7), U6.6 (PA4)
- new net: J2.8 (P8), U6.7 (PA5)
- new net: J2.9 (P9), U6.8 (PA6)
- new net: J2.10 (P10), U6.9 (PA7)
- new net A0: U6.38 (RS0), U7.10 (A0)
- new net A1: U6.37 (RS1), U7.9 (A1)
- new net A2: U6.36 (RS2), U7.8 (A2)
- new net A3: U6.35 (RS3), U7.7 (A3)
- new net A4: U7.6 (A4)
- new net CLK: U6.25 (PHI2)
- new net D0: U6.33 (D0), U7.11 (D0)
- new net D1: U6.32 (D1), U7.12 (D1)
- new net D2: U6.31 (D2), U7.13 (D2)
- new net D3: U6.30 (D3), U7.15 (D3)
- new net D4: U6.29 (D4), U7.16 (D4)
- new net D5: U6.28 (D5), U7.17 (D5)
- new net D6: U6.27 (D6), U7.18 (D6)
- new net D7: U6.26 (D7), U7.19 (D7)
- new net GND: J2.1 (P1), J2.2 (P2), J3.1 (P1), J3.2 (P2), U7.14 (GND), U7.21 (GND)
- new net R/~W: U6.22 (R/~W)
- new net VCC: J2.13 (P13), J2.14 (P14), J3.13 (P13), J3.14 (P14), U6.24 (CS1), U7.28 (VCC)
- new net ~7FAX: U7.20 (~CE)
- new net ~7FCX: U6.23 (~CS2)
- new net ~IRQ: D1.2 (A), U7.5 (~IRQ)
- new net ~MRD: U7.22 (~OE)
- new net ~MWR: U7.27 (~WE)
- new net ~PWR: U7.1 (~PWR)
- new net ~RES: U6.34 (~RESET), U7.4 (~RST)
- no-connect marks 0 -> 3
Other:
- note added: "The intention is to use a WDC65C22\nso a diod has been added."

Commit message: The PCB layout editor doesn't like 7805's footprint.
Parts:
- D1: footprint (none) -> Diodes_ThroughHole:D_DO-35_SOD27_P7.62mm_Horizontal
- J2, J3: footprint (none) -> Pin_Headers:Pin_Header_Straight_2x07_Pitch2.54mm
- U6: footprint (none) -> Housings_DIP:DIP-40_W15.24mm
- U7: footprint (none) -> Housings_DIP:DIP-28_W15.24mm
Connections:
- net GND: now also U6.1 (GND)
- net VCC: now also U6.20 (VCC)
