File: HW/IDE_interface/IDE_interface.sch (KiCad schematic (older format))
At the start: 16 parts, among them P1 EXPANSION PORT, P2 IDE0, U1 74LS32, U2 74LS139, U3 74HC74, U4 74LS08, U5 DS1511Y+, U6 74LS574, U7 74LS574, U8 74HC245

Commit message: New MB design. Includes RTC. New IDE design.
Parts:
- removed R4: 3.3K, Resistors_ThroughHole:Resistor_Horizontal_RM7mm, symbol R
- removed U5: DS1511Y+, Housings_DIP:DIP-28_W15.24mm, symbol DS1511Y+
- D1: footprint LEDs:LED-3MM -> LEDs:LED_D3.0mm
- P1: footprint Pin_Headers:Pin_Header_Straight_2x25 -> Pin_Headers:Pin_Header_Straight_2x25_Pitch2.54mm
- P2: footprint Pin_Headers:Pin_Header_Straight_2x20 -> Pin_Headers:Pin_Header_Straight_2x20_Pitch2.54mm
- R1, R2, R3, R5: footprint Resistors_ThroughHole:Resistor_Horizontal_RM7mm -> Resistors_ThroughHole:R_Axial_DIN0411_L9.9mm_D3.6mm_P12.70mm_Horizontal
- U1, U3: footprint Housings_DIP:DIP-14_W7.62mm -> Housings_DIP:DIP-14_W7.62mm_Socket
- U2: footprint Housings_DIP:DIP-16_W7.62mm -> Housings_DIP:DIP-16_W7.62mm_Socket
- U4: footprint Housings_DIP:DIP-8_W7.62mm -> Housings_DIP:DIP-8_W7.62mm_Socket
- U5: renamed from U6; footprint Housings_DIP:DIP-20_W7.62mm -> Housings_DIP:DIP-20_W7.62mm_Socket
- U6: renamed from U7; footprint Housings_DIP:DIP-20_W7.62mm -> Housings_DIP:DIP-20_W7.62mm_Socket
- U7: renamed from U8; footprint Housings_DIP:DIP-20_W7.62mm -> Housings_DIP:DIP-20_W7.62mm_Socket

Commit message: Updates to pcb and monitor.
Parts:
- P1: footprint Pin_Headers:Pin_Header_Straight_2x25_Pitch2.54mm -> Connect:IDC_Header_Straight_50pins
- P2: footprint Pin_Headers:Pin_Header_Straight_2x20_Pitch2.54mm -> Connect:IDC_Header_Straight_40pins
Changed lines of the file:
@@
 F 0 "P2" H 15000 2900 50  0000 C CNN
 F 1 "IDE0" V 15000 1850 50  0000 C CNN
-F 2 "Pin_Headers:Pin_Header_Straight_2x20_Pitch2.54mm" H 15000 900 50  0001 C CNN
+F 2 "Connect:IDC_Header_Straight_40pins" H 15000 900 50  0001 C CNN
 F 3 "" H 15000 900 50  0000 C CNN
 	1    15000 1850
@@
 F 0 "P1" H 3900 9900 50  0000 C CNN
 F 1 "EXPANSION PORT" V 3900 8600 50  0000 C CNN
-F 2 "Pin_Headers:Pin_Header_Straight_2x25_Pitch2.54mm" H 3900 7850 50  0001 C CNN
+F 2 "Connect:IDC_Header_Straight_50pins" H 3900 7850 50  0001 C CNN
 F 3 "" H 3900 7850 50  0000 C CNN
 	1    3900 8600
