File: HW/SBC/_saved_cpu_rom_ram.sch (KiCad schematic (older format))
At the start: 6 parts, among them U1 WD65C02_, U2 28C256, U3 HM62256BLP-7

Commit message: New SBC PCB. Started to split pluto_kernel.asm into bios, monitor and miniassembler/disassembler. Various other updates.
Changed lines of the file:
@@
 Connection ~ 4050 3000
 $Comp
-L GND #PWR?
+L GND #PWR01
 U 1 1 5924D5BB
 P 1525 3350
-F 0 "#PWR?" H 1525 3100 50  0001 C CNN
+F 0 "#PWR01" H 1525 3100 50  0001 C CNN
 F 1 "GND" H 1525 3225 50  0000 C CNN
 F 2 "" H 1525 3350 50  0001 C CNN
@@
 $EndComp
 $Comp
-L VCC #PWR?
+L VCC #PWR02
 U 1 1 5924D609
 P 1150 3250
-F 0 "#PWR?" H 1150 3100 50  0001 C CNN
+F 0 "#PWR02" H 1150 3100 50  0001 C CNN
 F 1 "VCC" H 1150 3400 50  0000 C CNN
 F 2 "" H 1150 3250 50  0001 C CNN
@@
 	0    -1   -1   0
 $EndComp
+$Comp
+L GND #PWR03
+U 1 1 5924DBE5
+P 5775 3550
+F 0 "#PWR03" H 5775 3300 50  0001 C CNN
+F 1 "GND" H 5775 3425 50  0000 C CNN
+F 2 "" H 5775 3550 50  0001 C CNN
+F 3 "" H 5775 3550 50  0001 C CNN
+	1    5775 3550
+	0    1    1    0
+$EndComp
+$Comp
+L VCC #PWR04
+U 1 1 5924DCC6
+P 5775 1050
+F 0 "#PWR04" H 5775 900 50  0001 C CNN
+F 1 "VCC" V 5700 1125 50  0000 C CNN
+F 2 "" H 5775 1050 50  0001 C CNN
+F 3 "" H 5775 1050 50  0001 C CNN
+	1    5775 1050
+	0    1    1    0
+$EndComp
+$Comp
+L VCC #PWR05
+U 1 1 5924DE07
+P 8475 1050
+F 0 "#PWR05" H 8475 900 50  0001 C CNN
+F 1 "VCC" H 8475 1200 50  0000 C CNN
+F 2 "" H 8475 1050 50  0001 C CNN
+F 3 "" H 8475 1050 50  0001 C CNN
+	1    8475 1050
+	1    0    0    -1
+$EndComp
+$Comp
+L GND #PWR06
+U 1 1 5924DE5C
+P 8475 3250
+F 0 "#PWR06" H 8475 3000 50  0001 C CNN
+F 1 "GND" H 8475 3125 50  0000 C CNN
+F 2 "" H 8475 3250 50  0001 C CNN
+F 3 "" H 8475 3250 50  0001 C CNN
+	1    8475 3250
+	0    1    1    0
+$EndComp
 $EndSCHEMATC
