File: HW/SBC/IDE16bit.sch (KiCad schematic (older format))
At the start: 13 parts, among them P1 IDE0, U16 74LS32, U17 74LS139, U18 74HC74, U19 74LS08, U20 74LS574, U21 74LS574, U22 74HC245

Commit message: Connected most hierarchical labels between the sheets. Added a connector to AY IO port.
Connections:
- net A3 renamed A[0..15]
- net CLK2 renamed CLK
- net ~7F8X renamed ~7F6X
Changed lines of the file:
@@
 $EndComp
 $Comp
-L GND #PWR52
+L GND #PWR053
 U 1 1 5932FB2C
 P 1350 950
-F 0 "#PWR52" H 1350 700 50  0001 C CNN
+F 0 "#PWR053" H 1350 700 50  0001 C CNN
 F 1 "GND" V 1350 775 50  0000 C CNN
 F 2 "" H 1350 950 50  0000 C CNN
@@
 $EndComp
 $Comp
-L VCC #PWR51
+L VCC #PWR054
 U 1 1 5932FB2D
 P 1325 1650
-F 0 "#PWR51" H 1325 1500 50  0001 C CNN
+F 0 "#PWR054" H 1325 1500 50  0001 C CNN
 F 1 "VCC" V 1325 1825 50  0000 C CNN
 F 2 "" H 1325 1650 50  0000 C CNN
@@
 $EndComp
 $Comp
-L VCC #PWR50
+L VCC #PWR055
 U 1 1 5932FB32
 P 800 8050
-F 0 "#PWR50" H 800 7900 50  0001 C CNN
+F 0 "#PWR055" H 800 7900 50  0001 C CNN
 F 1 "VCC" H 800 8200 50  0000 C CNN
 F 2 "" H 800 8050 50  0000 C CNN
@@
 NoConn ~ 4700 1500
 $Comp
-L GND #PWR53
+L GND #PWR056
 U 1 1 5932FB35
 P 2150 6050
-F 0 "#PWR53" H 2150 5800 50  0001 C CNN
+F 0 "#PWR056" H 2150 5800 50  0001 C CNN
 F 1 "GND" H 2150 5900 50  0000 C CNN
 F 2 "" H 2150 6050 50  0000 C CNN
@@
 Text Label 7725 9950 0    60   ~ 0
 ~IRQ
-Text Label 7725 10050 0    60   ~ 0
+Text Label 7050 10050 0    60   ~ 0
 A1
-Text Label 7725 10150 0    60   ~ 0
+Text Label 7050 10150 0    60   ~ 0
 A0
 Text Label 9125 10150 2    60   ~ 0
@@
 CLK2
 Text Label 1100 3100 0    60   ~ 0
-~7F8X
+~7F6X
 Text Label 1100 4100 0    60   ~ 0
 ~MWR
@@
 	8125 9850 7575 9850
 Wire Wire Line
-	8125 10050 7725 10050
-Wire Wire Line
-	8125 10150 7725 10150
+	8125 10050 7050 10050
+Wire Wire Line
+	8125 10150 7050 10150
 Wire Wire Line
 	8125 10250 7725 10250
@@
 	8625 9250 9125 9250
 Wire Wire Line
-	8625 9450 9125 9450
-Wire Wire Line
-	8625 9550 9125 9550
-Wire Wire Line
-	8625 9650 9125 9650
-Wire Wire Line
-	8625 9850 9125 9850
+	8625 9450 9400 9450
+Wire Wire Line
+	8625 9550 9400 9550
+Wire Wire Line
+	9400 9650 8625 9650
+Wire Wire Line
+	9400 9850 8625 9850
 Wire Wire Line
 	8625 10150 9125 10150
@@
 	8625 10250 9125 10250
 Wire Wire Line
-	8625 10350 9125 10350
+	9400 10350 8625 10350
 Wire Wire Line
 	8625 8450 9125 8450
@@
 	7050 9950 8125 9950
 Wire Wire Line
-	8625 9950 9125 9950
+	9400 9950 8625 9950
 Entry Wire Line
 	13575 2400 13675 2500
@@
 	13875 3300 13075 3300
 $Comp
-L GND #PWR?
+L GND #PWR057
 U 1 1 5933B988
 P 9125 8450
-F 0 "#PWR?" H 9125 8200 50  0001 C CNN
+F 0 "#PWR057" H 9125 8200 50  0001 C CNN
 F 1 "GND" H 9125 8300 50  0000 C CNN
 F 2 "" H 9125 8450 50  0001 C CNN
@@
 $EndComp
 $Comp
-L GND #PWR?
+L GND #PWR058
 U 1 1 5933C0BC
 P 7725 9350
-F 0 "#PWR?" H 7725 9100 50  0001 C CNN
+F 0 "#PWR058" H 7725 9100 50  0001 C CNN
 F 1 "GND" H 7725 9200 50  0000 C CNN
 F 2 "" H 7725 9350 50  0001 C CNN
@@
 Text HLabel 7050 9950 0    60   Input ~ 0
 ~IRQ
+$Comp
+L GND #PWR059
+U 1 1 5934CB71
+P 9400 10350
+F 0 "#PWR059" H 9400 10100 50  0001 C CNN
+F 1 "GND" H 9400 10200 50  0000 C CNN
+F 2 "" H 9400 10350 50  0001 C CNN
+F 3 "" H 9400 10350 50  0001 C CNN
+	1    9400 10350
+	1    0    0    -1
+$EndComp
+Wire Wire Line
+	9400 9450 9400 10350
+Connection ~ 9400 9950
+Connection ~ 9400 9850
+Connection ~ 9400 9650
+Connection ~ 9400 9550
+Text HLabel 1100 1100 0    60   Input ~ 0
+A[0..15]
+Text HLabel 1100 1950 0    60   Input ~ 0
+CLK
+Text HLabel 1100 2250 0    60   Input ~ 0
+~MRD
+Text HLabel 1100 3100 0    60   Input ~ 0
+~7F6X
+Text HLabel 1100 4100 0    60   Input ~ 0
+~MWR
+Entry Wire Line
+	6950 10250 7050 10150
+Entry Wire Line
+	6950 10150 7050 10050
+Wire Bus Line
+	6950 10150 6950 10250
+Wire Bus Line
+	6950 10250 6475 10250
+Text Label 6475 10250 0    60   ~ 0
+A[0..15]
+Text HLabel 6475 10250 0    60   Input ~ 0
+A[0..15]
 $EndSCHEMATC

Commit message: Still no VCC net in PCBnew.
Parts:
- removed D3: LED, LEDs:LED_D3.0mm, symbol LED-RESCUE-IDE_interface
- added D3: LED, LEDs:LED_D3.0mm, symbol LED
- U19: footprint Housings_DIP:DIP-8_W7.62mm_Socket -> Housings_DIP:DIP-14_W7.62mm_Socket
Connections:
- net ~IDE:DASP: now also D3.1 (K)
- net at R8.1: now also D3.2 (A)
Changed lines of the file:
@@
 EESchema Schematic File Version 2
-LIBS:pluto-rescue
 LIBS:power
 LIBS:device
@@
 LIBS:pluto
 LIBS:pluto-cache
-LIBS:IDE_interface-cache
 EELAYER 25 0
 EELAYER END
@@
 F 0 "U19" H 7550 2600 50  0000 C CNN
 F 1 "74LS08" H 7550 2500 50  0000 C CNN
-F 2 "Housings_DIP:DIP-8_W7.62mm_Socket" H 7550 2550 50  0001 C CNN
+F 2 "Housings_DIP:DIP-14_W7.62mm_Socket" H 7550 2550 50  0001 C CNN
 F 3 "" H 7550 2550 50  0000 C CNN
 	2    7550 2550
@@
 $EndComp
 $Comp
-L GND #PWR053
+L GND #PWR051
 U 1 1 5932FB2C
 P 1350 950
-F 0 "#PWR053" H 1350 700 50  0001 C CNN
+F 0 "#PWR051" H 1350 700 50  0001 C CNN
 F 1 "GND" V 1350 775 50  0000 C CNN
 F 2 "" H 1350 950 50  0000 C CNN
@@
 $EndComp
 $Comp
-L VCC #PWR054
+L VCC #PWR052
 U 1 1 5932FB2D
 P 1325 1650
-F 0 "#PWR054" H 1325 1500 50  0001 C CNN
+F 0 "#PWR052" H 1325 1500 50  0001 C CNN
 F 1 "VCC" V 1325 1825 50  0000 C CNN
 F 2 "" H 1325 1650 50  0000 C CNN
@@
 $EndComp
 $Comp
-L VCC #PWR055
+L VCC #PWR053
 U 1 1 5932FB32
 P 800 8050
-F 0 "#PWR055" H 800 7900 50  0001 C CNN
+F 0 "#PWR053" H 800 7900 50  0001 C CNN
 F 1 "VCC" H 800 8200 50  0000 C CNN
 F 2 "" H 800 8050 50  0000 C CNN
@@
 F 0 "U19" H 6000 2500 50  0000 C CNN
 F 1 "74LS08" H 6000 2400 50  0000 C CNN
-F 2 "Housings_DIP:DIP-8_W7.62mm_Socket" H 6000 2450 50  0001 C CNN
+F 2 "Housings_DIP:DIP-14_W7.62mm_Socket" H 6000 2450 50  0001 C CNN
 F 3 "" H 6000 2450 50  0000 C CNN
 	1    6000 2450
 	1    0    0    -1
-$EndComp
-$Comp
-L LED-RESCUE-IDE_interface D3
-U 1 1 5932FB34
-P 1500 8650
-F 0 "D3" H 1500 8750 50  0000 C CNN
-F 1 "LED" H 1500 8550 50  0000 C CNN
-F 2 "LEDs:LED_D3.0mm" H 1500 8650 50  0001 C CNN
-F 3 "" H 1500 8650 50  0000 C CNN
-	1    1500 8650
-	-1   0    0    1
 $EndComp
 NoConn ~ 4700 5700
@@
 NoConn ~ 4700 1500
 $Comp
-L GND #PWR056
+L GND #PWR054
 U 1 1 5932FB35
 P 2150 6050
-F 0 "#PWR056" H 2150 5800 50  0001 C CNN
+F 0 "#PWR054" H 2150 5800 50  0001 C CNN
 F 1 "GND" H 2150 5900 50  0000 C CNN
 F 2 "" H 2150 6050 50  0000 C CNN
@@
 	1200 8650 1300 8650
 Wire Wire Line
-	1700 8650 2100 8650
+	1600 8650 2100 8650
 Wire Wire Line
 	4700 5500 11700 5500
@@
 	13875 3300 13075 3300
 $Comp
-L GND #PWR057
+L GND #PWR055
 U 1 1 5933B988
 P 9125 8450
-F 0 "#PWR057" H 9125 8200 50  0001 C CNN
+F 0 "#PWR055" H 9125 8200 50  0001 C CNN
 F 1 "GND" H 9125 8300 50  0000 C CNN
 F 2 "" H 9125 8450 50  0001 C CNN
@@
 $EndComp
 $Comp
-L GND #PWR058
+L GND #PWR056
 U 1 1 5933C0BC
 P 7725 9350
-F 0 "#PWR058" H 7725 9100 50  0001 C CNN
+F 0 "#PWR056" H 7725 9100 50  0001 C CNN
 F 1 "GND" H 7725 9200 50  0000 C CNN
 F 2 "" H 7725 9350 50  0001 C CNN
@@
 ~IRQ
 $Comp
-L GND #PWR059
+L GND #PWR057
 U 1 1 5934CB71
 P 9400 10350
-F 0 "#PWR059" H 9400 10100 50  0001 C CNN
+F 0 "#PWR057" H 9400 10100 50  0001 C CNN
 F 1 "GND" H 9400 10200 50  0000 C CNN
 F 2 "" H 9400 10350 50  0001 C CNN
@@
 Text HLabel 6475 10250 0    60   Input ~ 0
 A[0..15]
+$Comp
+L LED D3
+U 1 1 59388E35
+P 1450 8650
+F 0 "D3" H 1450 8750 50  0000 C CNN
+F 1 "LED" H 1450 8550 50  0000 C CNN
+F 2 "LEDs:LED_D3.0mm" H 1450 8650 50  0001 C CNN
+F 3 "" H 1450 8650 50  0001 C CNN
+	1    1450 8650
+	-1   0    0    1
+$EndComp
 $EndSCHEMATC
