File: HW/SBC/audio.sch (KiCad schematic (older format))
At the start: 15 parts, among them J6 AY-IO, U13 LM386, U14 AY-3-8912

Commit message: Small changes to schematics. Futher development of BIOS.
Parts:
- removed C18: 10uF, Capacitors_ThroughHole:C_Disc_D3.8mm_W2.6mm_P2.50mm, symbol C_Small
- added C18: 10uF, symbol CP1_Small
Connections:
- net GND: now also C18.2
- net VCC: now also C18.1
Changed lines of the file:
@@
 LIBS:transistor
 LIBS:uln-ic
-LIBS:IDE_interface
+LIBS:+1.8V
+LIBS:+3.3V
+LIBS:+5V
+LIBS:+9V
+LIBS:25AA02EXXX-XOT
+LIBS:74LVC8T245
+LIBS:4021
+LIBS:7408
+LIBS:74125
+LIBS:74138
+LIBS:74148
+LIBS:74151
+LIBS:74157
+LIBS:74541
+LIBS:ANT
+LIBS:AP6502
+LIBS:AUDIO-JACK-3
+LIBS:AUDIO-JACK-6
+LIBS:BATTERY
+LIBS:BELFUSE-08B0-1X1T-06-F
+LIBS:C
+LIBS:CP
+LIBS:CRYSTAL
+LIBS:CRYSTAL-14
+LIBS:CVAR
+LIBS:DIODE
+LIBS:DIODES-AP3211
+LIBS:DIODESCH
+LIBS:DIODEZENER
+LIBS:DMMT5401
+LIBS:EDISON-BULB-E10
+LIBS:EDISON-SOCKET-E10
+LIBS:ENC28J60
+LIBS:FTDI-PLUG
+LIBS:GNDPWR
+LIBS:~GNDPWR
+LIBS:INDUCTOR
+LIBS:INTEL-EDISON-COMPUTE-MODULE
+LIBS:IS31AP4066D
+LIBS:JTAG
+LIBS:JTAG10
+LIBS:LATTICE-LC4256
+LIBS:LED
+LIBS:LED-BI
+LIBS:LED-BI-COMMON-CATHODE
+LIBS:LM324
+LIBS:LM1875
+LIBS:MAX3221
+LIBS:MC33926
+LIBS:MC34063A
+LIBS:MCP49X1
+LIBS:MCP3204
+LIBS:MECH
+LIBS:MIC2039
+LIBS:MIC2288
+LIBS:MICROSD-AMPHENOL-114-00841-68
+LIBS:MOSFET-N
+LIBS:MOSFET-N-123
+LIBS:MOSFET-N-134
+LIBS:MOSFET-P
+LIBS:NPN
+LIBS:nRF8001
+LIBS:NXPUDA1334ATS
+LIBS:OPAMP-DUAL
+LIBS:P01
+LIBS:P02
+LIBS:P03
+LIBS:P05
+LIBS:P06
+LIBS:P06-MOTOR
+LIBS:P08
+LIBS:P10
+LIBS:P22
+LIBS:P24
+LIBS:PHOTO_TRANSISTOR
+LIBS:PIEZO
+LIBS:PNP
+LIBS:POLYFUSE
+LIBS:POT
+LIBS:PWR_FLAG
+LIBS:QRE1113
+LIBS:R
+LIBS:RASPBERRYPI
+LIBS:RASPBERRYPI2
+LIBS:RBUS8
+LIBS:RN4020
+LIBS:ROBOT-P10-IO
+LIBS:RS-232-DB-9-DTE
+LIBS:SEN-SHT3x-DIS
+LIBS:SERVO
+LIBS:SI4737-C40-GM
+LIBS:SI4737-GU
+LIBS:SKYWORKS-AAT1217-3.3
+LIBS:SPDT
+LIBS:SPST
+LIBS:SPST-4PIN
+LIBS:SST25VF032B-S2A
+LIBS:SST26VF032B
+LIBS:ST-LIS3MDL
+LIBS:STM32-32PIN
+LIBS:STM32-48PIN
+LIBS:STM32-64PIN
+LIBS:STM32SWDUART
+LIBS:ST-SWD
+LIBS:ST-TDA7266
+LIBS:SWD
+LIBS:TCS3472
+LIBS:TI-ADS7866
+LIBS:TICC3000
+LIBS:TIREF30XX
+LIBS:TP
+LIBS:TS5A623157
+LIBS:TSV631
+LIBS:TVS-DIODE
+LIBS:TXB0108-PW
+LIBS:USBAB
+LIBS:Vcc
+LIBS:Vdd
+LIBS:VIN
+LIBS:VREG
+LIBS:VREG_VOUTCENTER
 LIBS:74xgxx
 LIBS:ac-dc
@@
 $EndComp
 $Comp
-L C_Small C18
-U 1 1 59307F3A
-P 2800 1125
-F 0 "C18" V 2675 1075 50  0000 L CNN
-F 1 "10uF" V 2925 1025 50  0000 L CNN
-F 2 "Capacitors_ThroughHole:C_Disc_D3.8mm_W2.6mm_P2.50mm" H 2800 1125 50  0001 C CNN
-F 3 "" H 2800 1125 50  0001 C CNN
-	1    2800 1125
-	0    1    1    0
-$EndComp
-$Comp
 L C_Small C20
 U 1 1 59307F57
@@
 Wire Wire Line
 	7125 2825 4950 2825
+$Comp
+L CP1_Small C18
+U 1 1 597D36E0
+P 2800 1125
+F 0 "C18" V 2925 1050 50  0000 L CNN
+F 1 "10uF" V 2675 1050 50  0000 L CNN
+F 2 "" H 2800 1125 50  0001 C CNN
+F 3 "" H 2800 1125 50  0001 C CNN
+	1    2800 1125
+	0    1    -1   0
+$EndComp
 $EndSCHEMATC
