File: SBC/power_and_expansion.sch (KiCad schematic (older format))
At the start: 8 parts, among them J4 BARREL_JACK, U11 LM7805CT

Commit message: Added dis-assembler. Removed files that was never needed. Updates to schematics files due to upgrade to KiCad 5.1.
Parts:
- C7, C8: symbol CP1_Small -> device:CP1_Small
- J4: symbol BARREL_JACK -> conn:BARREL_JACK
- MK3, MK4, MK5, MK6: symbol Mounting_Hole -> mechanical:Mounting_Hole
- U11: symbol LM7805CT-RESCUE-pluto -> pluto-rescue:LM7805CT-RESCUE-pluto
